File: VDD.kicad_sch (KiCad schematic)
At the start: 29 parts, among them IC1 TPS63070RNMR, J1 USB_B_Mini, J2 Jack-DC

Commit message: Adjusted the VDD supply schematic
Parts:
- removed C16: 100nF, symbol Device:C
- removed C16: 10uF, symbol Device:C
- added C16: 100nF, symbol Device:C
Connections:
- net GND: now also J1.2 (D-), J1.3 (D+), J1.4 (ID), C16.1
- net at IC1.3 (VAUX): now also C16.2
- no-connect marks 4 -> 1
Other:
- title: Component Supply -> (none)
- moved on the sheet: C17, R4, R7
