File: KiCad/VDD.kicad_sch (KiCad schematic)
At the start: 29 parts, among them IC1 TPS63070RNMR, J1 USB_B_Mini, J2 Jack-DC

Commit message: Pulling
Connections:
- net PS/S is gone; now on net GND: IC1.1 (PS/S), IC1.14 (EN), R4.1
Other:
- moved on the sheet: C16, R7
Changed lines of the file:
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@@
   (junction (at 96.52 129.54) (diameter 0) (color 0 0 0 0)
   )
+  (junction (at 76.2 137.16) (diameter 0) (color 0 0 0 0)
+  )
   (junction (at 91.44 177.8) (diameter 0) (color 0 0 0 0)
   )
@@
   (junction (at 111.76 129.54) (diameter 0) (color 0 0 0 0)
   )
-  (junction (at 85.09 129.54) (diameter 0) (color 0 0 0 0)
+  (junction (at 86.36 129.54) (diameter 0) (color 0 0 0 0)
   )
   (junction (at 86.36 38.1) (diameter 0) (color 0 0 0 0)
@@
   (junction (at 116.84 38.1) (diameter 0) (color 0 0 0 0)
   )
-  (junction (at 26.67 127) (diameter 0) (color 0 0 0 0)
+  (junction (at 27.94 127) (diameter 0) (color 0 0 0 0)
   )
   (junction (at 22.86 30.48) (diameter 0) (color 0 0 0 0)
@@
     (stroke (width 0) (type default))
   )
-  (wire (pts (xy 38.1 118.11) (xy 38.1 124.46))
+  (wire (pts (xy 38.1 119.38) (xy 38.1 124.46))
     (stroke (width 0) (type default))
   )
@@
     (stroke (width 0) (type default))
   )
-  (wire (pts (xy 24.13 127) (xy 26.67 127))
+  (wire (pts (xy 25.4 127) (xy 27.94 127))
     (stroke (width 0) (type default))
   )
@@
     (stroke (width 0) (type default))
   )
-  (wire (pts (xy 76.2 135.89) (xy 81.28 135.89))
+  (wire (pts (xy 76.2 137.16) (xy 81.28 137.16))
     (stroke (width 0) (type default))
   )
@@
     (stroke (width 0) (type default))
   )
-  (wire (pts (xy 81.28 135.89) (xy 81.28 142.24))
+  (wire (pts (xy 81.28 137.16) (xy 81.28 142.24))
     (stroke (width 0) (type default))
   )
@@
     (stroke (width 0) (type default))
   )
-  (wire (pts (xy 43.18 129.54) (xy 26.67 129.54))
+  (wire (pts (xy 43.18 129.54) (xy 27.94 129.54))
     (stroke (width 0) (type default))
   )
@@
     (stroke (width 0) (type default))
   )
-  (wire (pts (xy 36.83 127) (xy 43.18 127))
+  (wire (pts (xy 38.1 127) (xy 43.18 127))
     (stroke (width 0) (type default))
   )
@@
     (stroke (width 0) (type default))
   )
-  (wire (pts (xy 35.56 118.11) (xy 38.1 118.11))
+  (wire (pts (xy 35.56 119.38) (xy 38.1 119.38))
     (stroke (width 0) (type default))
   )
@@
     (stroke (width 0) (type default))
   )
-  (wire (pts (xy 26.67 127) (xy 26.67 129.54))
+  (wire (pts (xy 27.94 127) (xy 27.94 129.54))
     (stroke (width 0) (type default))
   )
@@
     (stroke (width 0) (type default))
   )
-  (wire (pts (xy 26.67 118.11) (xy 27.94 118.11))
-    (stroke (width 0) (type default))
-  )
   (wire (pts (xy 30.48 66.04) (xy 38.1 66.04))
     (stroke (width 0) (type default))
@@
     (stroke (width 0) (type default))
   )
-  (wire (pts (xy 76.2 135.89) (xy 76.2 134.62))
+  (wire (pts (xy 76.2 137.16) (xy 76.2 134.62))
     (stroke (width 0) (type default))
   )
@@
     (stroke (width 0) (type default))
   )
-  (wire (pts (xy 78.74 129.54) (xy 85.09 129.54))
-    (stroke (width 0) (type default))
-  )
-  (wire (pts (xy 85.09 129.54) (xy 96.52 129.54))
+  (wire (pts (xy 78.74 129.54) (xy 86.36 129.54))
+    (stroke (width 0) (type default))
+  )
+  (wire (pts (xy 86.36 129.54) (xy 96.52 129.54))
     (stroke (width 0) (type default))
   )
@@
     (stroke (width 0) (type default))
   )
-  (wire (pts (xy 26.67 127) (xy 29.21 127))
+  (wire (pts (xy 27.94 127) (xy 30.48 127))
     (stroke (width 0) (type default))
   )
@@
     )
   )
-  (global_label "PG" (shape input) (at 80.01 177.8 90) (fields_autoplaced)
+  (global_label "PG" (shape input) (at 81.28 177.8 90) (fields_autoplaced)
     (effects (font (size 1.27 1.27)) (justify left))
-    (property "Intersheetrefs" "${INTERSHEET_REFS}" (at 80.01 172.3542 90)
+    (property "Intersheetrefs" "${INTERSHEET_REFS}" (at 81.28 172.3542 90)
       (effects (font (size 1.27 1.27)) (justify left) hide)
     )
@@
     )
   )
-  (global_label "PG" (shape input) (at 26.67 118.11 180) (fields_autoplaced)
+  (global_label "PG" (shape input) (at 27.94 119.38 180) (fields_autoplaced)
     (effects (font (size 1.27 1.27)) (justify right))
-    (property "Intersheetrefs" "${INTERSHEET_REFS}" (at 21.2242 118.11 0)
+    (property "Intersheetrefs" "${INTERSHEET_REFS}" (at 22.4942 119.38 0)
       (effects (font (size 1.27 1.27)) (justify right) hide)
     )
@@
     )
   )
-  (symbol (lib_id "power:GND") (at 24.13 127 270) (unit 1)
-    (in_bom yes) (on_board yes) (dnp no) (fields_autoplaced)
-    (property "Reference" "#PWR019" (at 17.78 127 0)
-      (effects (font (size 1.27 1.27)) hide)
-    )
-    (property "Value" "GND" (at 20.32 127.635 90)
+  (symbol (lib_id "power:GND") (at 25.4 127 270) (unit 1)
+    (in_bom yes) (on_board yes) (dnp no) (fields_autoplaced)
+    (property "Reference" "#PWR019" (at 19.05 127 0)
+      (effects (font (size 1.27 1.27)) hide)
+    )
+    (property "Value" "GND" (at 21.59 127.635 90)
       (effects (font (size 1.27 1.27)) (justify right))
     )
-    (property "Footprint" "" (at 24.13 127 0)
-      (effects (font (size 1.27 1.27)) hide)
-    )
-    (property "Datasheet" "" (at 24.13 127 0)
+    (property "Footprint" "" (at 25.4 127 0)
+      (effects (font (size 1.27 1.27)) hide)
+    )
+    (property "Datasheet" "" (at 25.4 127 0)
       (effects (font (size 1.27 1.27)) hide)
     )
@@
     )
   )
-  (symbol (lib_id "Device:R") (at 31.75 118.11 270) (unit 1)
+  (symbol (lib_id "Device:R") (at 31.75 119.38 270) (unit 1)
     (in_bom yes) (on_board yes) (dnp no)
-    (property "Reference" "R7" (at 31.75 120.65 90)
-      (effects (font (size 1.27 1.27)))
-    )
-    (property "Value" "100K" (at 31.75 115.57 90)
-      (effects (font (size 1.27 1.27)))
-    )
-    (property "Footprint" "" (at 31.75 116.332 90)
-      (effects (font (size 1.27 1.27)) hide)
-    )
-    (property "Datasheet" "~" (at 31.75 118.11 0)
+    (property "Reference" "R7" (at 31.75 121.92 90)
+      (effects (font (size 1.27 1.27)))
+    )
+    (property "Value" "100K" (at 31.75 116.84 90)
+      (effects (font (size 1.27 1.27)))
+    )
+    (property "Footprint" "" (at 31.75 117.602 90)
+      (effects (font (size 1.27 1.27)) hide)
+    )
+    (property "Datasheet" "~" (at 31.75 119.38 0)
       (effects (font (size 1.27 1.27)) hide)
     )
@@
     )
   )
-  (symbol (lib_id "power:GND") (at 85.09 137.16 0) (unit 1)
+  (symbol (lib_id "power:GND") (at 86.36 137.16 0) (unit 1)
     (in_bom yes) (on_board yes) (dnp no)
-    (property "Reference" "#PWR018" (at 85.09 143.51 0)
-      (effects (font (size 1.27 1.27)) hide)
-    )
-    (property "Value" "GND" (at 85.09 137.16 0)
-      (effects (font (size 1.27 1.27)))
-    )
-    (property "Footprint" "" (at 85.09 137.16 0)
-      (effects (font (size 1.27 1.27)) hide)
-    )
-    (property "Datasheet" "" (at 85.09 137.16 0)
+    (property "Reference" "#PWR018" (at 86.36 143.51 0)
+      (effects (font (size 1.27 1.27)) hide)
+    )
+    (property "Value" "GND" (at 86.36 137.16 0)
+      (effects (font (size 1.27 1.27)))
+    )
+    (property "Footprint" "" (at 86.36 137.16 0)
+      (effects (font (size 1.27 1.27)) hide)
+    )
+    (property "Datasheet" "" (at 86.36 137.16 0)
       (effects (font (size 1.27 1.27)) hide)
     )
@@
     )
   )
-  (symbol (lib_id "Device:C") (at 33.02 127 90) (unit 1)
+  (symbol (lib_id "Device:C") (at 34.29 127 90) (unit 1)
     (in_bom yes) (on_board yes) (dnp no)
-    (property "Reference" "C16" (at 35.56 125.73 90)
-      (effects (font (size 1.27 1.27)))
-    )
-    (property "Value" "100nF" (at 27.94 125.73 90)
-      (effects (font (size 1.27 1.27)))
-    )
-    (property "Footprint" "" (at 36.83 126.0348 0)
-      (effects (font (size 1.27 1.27)) hide)
-    )
-    (property "Datasheet" "~" (at 33.02 127 0)
+    (property "Reference" "C16" (at 36.83 125.73 90)
+      (effects (font (size 1.27 1.27)))
+    )
+    (property "Value" "100nF" (at 29.21 125.73 90)
+      (effects (font (size 1.27 1.27)))
+    )
+    (property "Footprint" "" (at 38.1 126.0348 0)
+      (effects (font (size 1.27 1.27)) hide)
+    )
+    (property "Datasheet" "~" (at 34.29 127 0)
       (effects (font (size 1.27 1.27)) hide)
     )
@@
     )
   )
-  (symbol (lib_id "Device:C") (at 85.09 133.35 0) (unit 1)
-    (in_bom yes) (on_board yes) (dnp no) (fields_autoplaced)
-    (property "Reference" "C16" (at 89.154 132.715 0)
-      (effects (font (size 1.27 1.27)) (justify left))
-    )
-    (property "Value" "10uF" (at 89.154 135.255 0)
-      (effects (font (size 1.27 1.27)) (justify left))
-    )
-    (property "Footprint" "" (at 86.0552 137.16 0)
-      (effects (font (size 1.27 1.27)) hide)
-    )
-    (property "Datasheet" "~" (at 85.09 133.35 0)
-      (effects (font (size 1.27 1.27)) hide)
-    )
+  (symbol (lib_id "Device:C") (at 86.36 133.35 0) (unit 1)
+    (in_bom yes) (on_board yes) (dnp no) (fields_autoplaced)
+    (property "Reference" "C16" (at 90.424 132.715 0)
+      (effects (font (size 1.27 1.27)) (justify left))
+    )
+    (property "Value" "10uF" (at 90.424 135.255 0)
+      (effects (font (size 1.27 1.27)) (justify left))
+    )
+    (property "Footprint" "" (at 87.3252 137.16 0)
+      (effects (font (size 1.27 1.27)) hide)
+    )
+    (property "Datasheet" "~" (at 86.36 133.35 0)
+      (effects (font (size 1.27 1.27)) hide)
+    )
