File: KiCad/Main_Supply.kicad_sch (KiCad schematic)
At the start: 20 parts, among them IC1 ISL23511WFB8Z, IC1 TPS63070RNMR, J1 USB_B_Mini, J2 Jack-DC, SW1 SW_Push

Commit message: Schematics updated. footprint assignment and layout still needed
Parts:
- removed D1, D2: D_Zener, symbol Device:D_Zener
- removed J1: USB_B_Mini, Connector_USB:USB_Micro-B_Molex_47346-0001, symbol Connector:USB_B_Mini
- removed J2: Jack-DC, symbol Connector:Jack-DC
Connections:
- net PG renamed VOUT
- no-connect marks 4 -> 0
Other:
- note removed: "Connectors"
