File: KiCad/MCU.kicad_sch (KiCad schematic)
At the start: 4 parts, among them SW1 SW_SPST, U1 STM32F401RBTx

Commit message: Schematic redesign needs two footprints before complete.
Parts:
- removed C9: 100nF, symbol Device:C
- removed R3: 1k, symbol Device:R
- removed SW1: SW_SPST, symbol Switch:SW_SPST
- removed U1: STM32F401RBTx, Package_QFP:LQFP-64_10x10mm_P0.5mm, symbol MCU_ST_STM32F4:STM32F401RBTx
