File: Power_Supply/Main_Supply.kicad_sch (KiCad schematic)
At the start: 20 parts, among them IC1 ISL23511WFB8Z, IC1 TPS63070RNMR, J1 USB_B_Mini, J2 Jack-DC, SW1 SW_Push

Commit message: Updated Schematic and VIM878
Parts:
- removed D1, D2: D_Zener, symbol Device:D_Zener
- removed J1: USB_B_Mini, Connector_USB:USB_Micro-B_Molex_47346-0001, symbol Connector:USB_B_Mini
- removed J2: Jack-DC, symbol Connector:Jack-DC
- C16, C17, C21: footprint (none) -> Capacitor_SMD:C_0805_2012Metric
- C16, C18, C19, C20: footprint (none) -> Capacitor_SMD:C_0402_1005Metric
- IC1: footprint SOIC127P600X175-8N -> Custom_eric:SOIC127P600X175-8N
- R4, R7: footprint (none) -> Resistor_SMD:R_0402_1005Metric
Connections:
- net PG renamed VOUT
- net VIN renamed Raw
- no-connect marks 4 -> 0
Other:
- note removed: "Connectors"
