File: Power_Supply/Main_output.kicad_sch (KiCad schematic)
At the start: 4 parts, among them J4 Conn_02x02_Odd_Even, J5 Conn_02x02_Odd_Even

Commit message: Updated Schematic and VIM878
Parts:
- J4, J5: footprint (none) -> Connector_PinHeader_2.54mm:PinHeader_2x02_P2.54mm_Vertical
- R11: value 300 -> 100; footprint (none) -> Resistor_SMD:R_0402_1005Metric
- R9: footprint (none) -> Resistor_SMD:R_0402_1005Metric
Connections:
- net GND: now also J4.2 (Pin_2), J4.4 (Pin_4), J5.2 (Pin_2), J5.4 (Pin_4); no longer J4.1 (Pin_1), J4.3 (Pin_3), J5.1 (Pin_1), J5.3 (Pin_3)
- net Main_Supply: now also J4.1 (Pin_1), J4.3 (Pin_3), J5.1 (Pin_1), J5.3 (Pin_3); no longer J4.2 (Pin_2), J4.4 (Pin_4), J5.2 (Pin_2), J5.4 (Pin_4)
