File: Power_Supply/Board_PWR.kicad_sch (KiCad schematic)
At the start: 21 parts, among them J1 USB_B_Mini, U3 LD3985G18R_TSOT23

Commit message: Kicad model updated.
Parts:
- added D3: LED, LED_SMD:LED_0603_1608Metric, symbol Device:LED
- added R1: 200, Resistor_SMD:R_0402_1005Metric, symbol Device:R
- D2: footprint (none) -> Diode_SMD:D_SOD-123
- FB1: footprint (none) -> Inductor_SMD:L_1206_3216Metric
Connections:
- net GND: now also C18.2, C19.2, C21.2, R1.2
- net board_out: now also D3.2 (A)
- net usb_out: now reaches D2.2 (A), J1.1 (VBUS)
- new net: D3.1 (K), R1.1
Other:
- moved on the sheet: C16, D2
