File: Power_Supply/VDD.kicad_sch (KiCad schematic)
At the start: 20 parts, among them IC1 ISL23511WFB8Z, IC1 TPS63070RNMR, SW1 SW_Push

Commit message: Kicad model updated.
Parts:
- removed C21 (x2): 10uF, Capacitor_SMD:C_0805_2012Metric, symbol Device:C
- removed R2, R3: 100, Resistor_SMD:R_0402_1005Metric, symbol Device:R
- added D1, D2: D_Zener, symbol Device:D_Zener
- added J1: USB_B_Mini, Connector_USB:USB_Micro-B_Molex_47346-0001, symbol Connector:USB_B_Mini
- added J2: Jack-DC, symbol Connector:Jack-DC
- C16, C17, C21: footprint Capacitor_SMD:C_0805_2012Metric -> (none)
- C16, C18, C19, C20: footprint Capacitor_SMD:C_0402_1005Metric -> (none)
- FB1: footprint Inductor_SMD:L_1206_3216Metric -> (none)
- IC1: footprint Custom_eric:SOIC127P600X175-8N -> SOIC127P600X175-8N
- L1: footprint Inductor_SMD:L_0603_1608Metric -> (none)
- R4, R7: footprint Resistor_SMD:R_0402_1005Metric -> (none)
Connections:
- net Pot_dwn is gone; now on an unnamed net: IC1.2 (~{PD})
- net Pot_up is gone; now on an unnamed net: IC1.1 (~{PU})
- net VOUT is gone; now on net PG: C19.1, C20.1, C21.1, FB1.2, IC1.3 (RH), IC1.7 (VOUT_1), IC1.8 (VOUT_2), R7.2
- net +3.3V: now also IC1.4 (VSS); no longer IC1.8 (VCC)
- net GND: now also IC1.8 (VCC), J1.5 (GND), J2.2; no longer IC1.4 (VSS)
- net Main_Supply: no longer C18.1
- net PG: now also C18.1; no longer IC1.2 (PG), R7.1
- net PS/S: now reaches IC1.1 (PS/S), IC1.14 (EN), R4.1
- net Raw renamed VIN
- net VIN: now also D1.1 (K), D2.1 (K)
- net switch_L1: no longer names the net of IC1.11 (L1), L1.2
- net switch_L2: no longer names the net of IC1.9 (L2), L1.1
- new net: D1.2 (A), J1.1 (VBUS)
- new net: IC1.2 (PG), R7.1
- new net: D2.2 (A), J2.1
- no-connect marks 0 -> 4
Other:
- note added: "Connectors"
- moved on the sheet: C16, C18, SW1
