File: Power_Supply/power_supply.kicad_pcb (KiCad board)
At the start: 2 copper layers, 5 parts, among them IC2 TPS63070RNMR, J1 USB_B_Mini, SW1 SW_Push, U1 STM32F401RBTx

Commit message: Kicad model updated.
Parts:
- removed J1: USB_B_Mini, Connector_USB:USB_Micro-B_Molex_47346-0001
- removed JP1: Jumper_2_Open, TestPoint:TestPoint_Bridge_Pitch2.54mm_Drill0.7mm
- removed SW1: SW_Push, Button_Switch_THT:SW_PUSH_6mm_H7.3mm
- added C1: 10uF, Capacitor_SMD:C_0805_2012Metric, F.Cu at (221.1, 72.9)
- added C10: 100nF, Capacitor_SMD:C_0402_1005Metric, F.Cu at (202.9, 71.2)
- added C11: 4uF7, Capacitor_SMD:C_0603_1608Metric, F.Cu at (199.7, 71.4)
- added C12: 100nF, Capacitor_SMD:C_0402_1005Metric, F.Cu at (182.7, 60.6)
- added C13: 100nF, Capacitor_SMD:C_0402_1005Metric, F.Cu at (196.5, 74.3)
- added C14: 16pF, Capacitor_SMD:C_0402_1005Metric, F.Cu at (188.7, 49.2)
- added C15: 16pF, Capacitor_SMD:C_0402_1005Metric, F.Cu at (181.7, 49.1)
- added C16: 4uF7, Capacitor_SMD:C_0603_1608Metric, F.Cu at (203.2, 74.0)
- added C17: 10nF, Capacitor_SMD:C_0805_2012Metric, F.Cu at (205.7, 40.4)
- added C18: 10uF, Capacitor_SMD:C_0805_2012Metric, F.Cu at (194.4, 87.8)
- added C19: 10uF, Capacitor_SMD:C_0805_2012Metric, F.Cu at (205.8, 44.4)
- added C2: 100nF, Capacitor_SMD:C_0402_1005Metric, F.Cu at (201.8, 80.3)
- added C20: 10uF, Capacitor_SMD:C_0805_2012Metric, F.Cu at (214.2, 44.7)
- added C21: 22uF, Capacitor_SMD:C_0402_1005Metric, F.Cu at (195.1, 47.9)
- added C22: 22uF, Capacitor_SMD:C_0402_1005Metric, F.Cu at (202.1, 42.0)
- added C23: 10uF, Capacitor_SMD:C_0805_2012Metric, F.Cu at (194.3, 91.4)
- added C24: 10uF, Capacitor_SMD:C_0805_2012Metric, F.Cu at (198.9, 42.7)
- added C25: 22uF, Capacitor_SMD:C_0402_1005Metric, F.Cu at (203.5, 110.0)
- added C27: 22uF, Capacitor_SMD:C_0402_1005Metric, F.Cu at (207.3, 100.3)
- added C29: 22uF, Capacitor_SMD:C_0402_1005Metric, F.Cu at (207.3, 102.9)
- added C3: 100nF, Capacitor_SMD:C_0402_1005Metric, F.Cu at (209.4, 61.0)
- added C31: 10uF, Capacitor_SMD:C_0805_2012Metric, F.Cu at (207.7, 97.8)
- added C34: 10uF, Capacitor_SMD:C_0805_2012Metric, F.Cu at (216.5, 72.9)
- added C35: 10uF, Capacitor_SMD:C_0805_2012Metric, F.Cu at (211.8, 73.0)
- added C4: 100nF, Capacitor_SMD:C_0402_1005Metric, F.Cu at (212.5, 61.0)
- added C5: 100nF, Capacitor_SMD:C_0402_1005Metric, F.Cu at (212.4, 56.8)
- added C6: 100nF, Capacitor_SMD:C_0402_1005Metric, F.Cu at (215.5, 56.7)
- added C7: 100nF, Capacitor_SMD:C_0402_1005Metric, F.Cu at (209.4, 56.8)
- added C8: 100nF, Capacitor_SMD:C_0402_1005Metric, F.Cu at (196.6, 71.2)
- added C9: 100nF, Capacitor_SMD:C_0402_1005Metric, F.Cu at (218.6, 56.8)
- added D1: D_Schottky, RB168VWM-30TR:RB168VWM30TR, F.Cu at (220.1, 41.4)
- added D2: D_Zener, Diode_SMD:D_SOD-123, F.Cu at (217.1, 45.4)
- added D3: LED, LED_SMD:LED_0603_1608Metric, F.Cu at (191.3, 42.4)
- added DWN: SW_Push, Button_Switch_THT:SW_PUSH_6mm_H7.3mm, F.Cu at (189.2, 99.2)
- added FB1: FerriteBead, Inductor_SMD:L_1206_3216Metric, F.Cu at (195.1, 43.3)
- added FB2: FerriteBead, Inductor_SMD:L_1206_3216Metric, F.Cu at (203.0, 105.6)
- added H1: MountingHole, MountingHole:MountingHole_2.1mm, F.Cu at (229.9, 50.4)
- added H2: MountingHole, MountingHole:MountingHole_2.1mm, F.Cu at (229.8, 106.5)
- added H3: MountingHole, MountingHole:MountingHole_2.1mm, F.Cu at (208.4, 50.4)
- added H4: MountingHole, MountingHole:MountingHole_2.1mm, F.Cu at (208.4, 106.2)
- added H5: MountingHole, MountingHole:MountingHole_3.2mm_M3, F.Cu at (229.8, 38.5)
- added H6: MountingHole, MountingHole:MountingHole_3.2mm_M3, F.Cu at (184.0, 38.6)
- added IC1: ISL23511WFB8Z, Custom_eric:SOIC127P600X175-8N, F.Cu at (206.4, 88.8)
- added J2: USB_B_Mini, Connector_USB:USB_Micro-B_Molex_47346-0001, F.Cu at (216.5, 34.4)
- added J3: Conn_01x05_Pin, Connector_JST:JST_EH_B5B-EH-A_1x05_P2.50mm_Vertical, F.Cu at (192.9, 34.7)
- added J4: Conn_02x02_Odd_Even, Connector_PinHeader_2.54mm:PinHeader_2x02_P2.54mm_Vertical, B.Cu at (228.9, 127.1)
- added J5: Conn_02x02_Odd_Even, Connector_PinHeader_2.54mm:PinHeader_2x02_P2.54mm_Vertical, B.Cu at (184.6, 126.9)
- added J6: Conn_01x04_Socket, Connector_PinSocket_2.54mm:PinSocket_1x04_P2.54mm_Vertical, F.Cu at (222.9, 63.5)
- added L2: 1.5uH, Inductor_SMD:L_0603_1608Metric, F.Cu at (211.6, 78.4)
- added R1: 200, Resistor_SMD:R_0402_1005Metric, F.Cu at (191.1, 45.7)
- added R10: 100K, Resistor_SMD:R_0402_1005Metric, F.Cu at (200.0, 77.1)
- added R11: 100, Resistor_SMD:R_0402_1005Metric, F.Cu at (193.6, 71.2)
- added R13: 10K, Resistor_SMD:R_0402_1005Metric, F.Cu at (207.8, 73.1)
- added R2: 100, Resistor_SMD:R_0402_1005Metric, F.Cu at (194.2, 84.7)
- added R3: 100, Resistor_SMD:R_0402_1005Metric, F.Cu at (194.3, 94.4)
- added R9: 100, Resistor_SMD:R_0402_1005Metric, F.Cu at (193.5, 74.2)
- added RST: SW_Push, Button_Switch_THT:SW_PUSH_6mm_H7.3mm, F.Cu at (189.3, 69.6)
- added U3: LD3985G18R_TSOT23, Package_TO_SOT_SMD:TSOT-23-5, F.Cu at (209.9, 42.1)
- added UP: SW_Push, Button_Switch_THT:SW_PUSH_6mm_H7.3mm, F.Cu at (182.8, 79.8)
- added Y1: 26MHz, Crystal:Crystal_SMD_ECS_CSM3X-2Pin_7.6x4.1mm, F.Cu at (184.8, 53.5)
- moved U1 64.0 mm to (198.9, 60.4)
- moved IC2 55.7 mm to (206.0, 78.4)
Connections:
- net PS/S renamed Net-(IC2-EN)
- net VDD renamed +3.3V
- IC2 pad 11: Net-(IC2-L1) -> /Main_Supply/switch_L1
- IC2 pad 12: VIN -> Raw
- IC2 pad 13: VIN -> Raw
- IC2 pad 16: (no net) -> Raw
- IC2 pad 17: (no net) -> VOUT
- IC2 pad 2: Net-(IC2-PG) -> /Main_Supply/PG
- IC2 pad 7: PG -> VOUT
- IC2 pad 8: PG -> VOUT
- IC2 pad 9: Net-(IC2-L2) -> /Main_Supply/switch_L2
- U1 pad 23: POT_UP -> unconnected-(U1-PA7-Pad23)
- U1 pad 24: POT_DWN -> unconnected-(U1-PC4-Pad24)
- U1 pad 27: BTN_UP -> unconnected-(U1-PB1-Pad27)
- U1 pad 28: BTN_DWN -> unconnected-(U1-PB2-Pad28)
- U1 pad 30: Net-(U1-VCAP1) -> /V_Cap
- U1 pad 5: Net-(U1-PH0) -> /Crystal_in
- U1 pad 6: Net-(U1-PH1) -> /Crystal_out
- U1 pad 60: Net-(JP1-B) -> GND
- U1 pad 7: Net-(U1-NRST) -> /Nrst
Routing:
- net GND: track 0.00 -> 164.1 mm, vias 0 -> 29
- net Main_Supply: track 0.00 -> 123.8 mm, vias 0 -> 2
- net +3.3V: track 0.00 -> 79.2 mm, vias 0 -> 7
- net Raw: track 0.00 -> 54.7 mm, vias 0 -> 2
- net VOUT: track 0.00 -> 51.8 mm, vias 0 -> 2
- net SDA: track 0.00 -> 28.8 mm, vias 0 -> 1
- net SWDIO: track 0.00 -> 28.0 mm, vias 0 -> 2
- net SCL: track 0.00 -> 25.1 mm, vias 0 -> 1
- net SWCLCK: track 0.00 -> 23.9 mm, vias 0 -> 1
- net /Nrst: track 0.00 -> 22.0 mm
- net SWO: track 0.00 -> 20.3 mm, vias 0 -> 1
- net /Crystal_out: track 0.00 -> 19.9 mm
- net /Main_Supply/Pot_dwn: track 0.00 -> 19.3 mm
- net /Main_Supply/Pot_up: track 0.00 -> 19.2 mm
- net board_out: track 0.00 -> 18.5 mm
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- added copper zone on In2.Cu, net +3.3V
- added copper zone on F.Cu, net /Board_PWR/usb_out
- added copper zone on B.Cu, net GND
- added copper zone on F.Cu, net Raw
Other:
- board outline added: 59.5 x 101.7 mm
- copper layers 2 -> 4
- board text added: "1"
- board text added: "SCL"
- board text added: "SDA"
- board text added: "SWCLCK"
- board text added: "SWDIO"
- board text added: "SWO"
- board text added: "VDD"
- board text added: "VSS"

Commit message: Updated schematics. and added the correct Driver files for stm32f401
Parts:
- moved R11 4.63 mm to (190.4, 74.5), turned to 90 degrees
- moved R9 0.34 mm to (193.4, 74.5), turned to 90 degrees
Routing:
- net Raw: track 54.7 -> 23.8 mm
- net GND: track 164.1 -> 137.8 mm, vias 29 -> 25
- net Main_Supply: track 123.8 -> 138.4 mm
- net VOUT: track 51.8 -> 53.1 mm
- net ADC1: track 16.4 -> 15.5 mm
- net SWCLCK: track 23.9 -> 24.7 mm
- net SWDIO: track 28.0 -> 28.7 mm
- added copper zone on F.Cu, net GND
- added copper zone on In1.Cu, net Raw
